File: Hardware/g081_audio/Euro.kicad_sch (KiCad schematic)
At the start: 67 parts, among them J10 AudioJack2_SwitchT, J4 AudioJack2_SwitchT, J5 AudioJack2_SwitchT, J6 AudioJack2_SwitchT, J7 AudioJack2_SwitchT, J8 Conn_02x08_Odd_Even, J9 AudioJack2_SwitchT, U10 LP2985-3.3, U6 LM4040DBZ-5, U7 MCP6004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

Commit message: Added schematic and more documentation.
Parts:
- R12, R13: value 33k -> 24.9k
Changed lines of the file:
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@@
 		)
 		(property "Intersheetrefs" "${INTERSHEET_REFS}"
-			(at 0 0 0)
+			(at 117.4776 40.64 0)
 			(effects
 				(font
 					(size 1.27 1.27)
 				)
+				(justify left)
 				(hide yes)
 			)
@@
 		)
 		(property "Intersheetrefs" "${INTERSHEET_REFS}"
-			(at 0 0 0)
+			(at 109.7367 234.95 0)
 			(effects
 				(font
 					(size 1.27 1.27)
 				)
+				(justify left)
 				(hide yes)
 			)
@@
 		)
 		(property "Intersheetrefs" "${INTERSHEET_REFS}"
-			(at 0 0 0)
+			(at 115.0586 85.09 0)
 			(effects
 				(font
 					(size 1.27 1.27)
 				)
+				(justify left)
 				(hide yes)
 			)
@@
 		)
 		(property "Intersheetrefs" "${INTERSHEET_REFS}"
-			(at 0 0 0)
+			(at 109.7367 185.42 0)
 			(effects
 				(font
 					(size 1.27 1.27)
 				)
+				(justify left)
 				(hide yes)
 			)
@@
 		)
 		(property "Intersheetrefs" "${INTERSHEET_REFS}"
-			(at 0 0 0)
+			(at 292.7325 40.64 0)
 			(effects
 				(font
 					(size 1.27 1.27)
 				)
+				(justify right)
 				(hide yes)
 			)
@@
 		)
 		(property "Intersheetrefs" "${INTERSHEET_REFS}"
-			(at 0 0 0)
+			(at 292.6115 85.09 0)
 			(effects
 				(font
 					(size 1.27 1.27)
 				)
+				(justify right)
 				(hide yes)
 			)
@@
 			)
 		)
-		(property "Value" "33k"
+		(property "Value" "24.9k"
 			(at 83.82 72.39 90)
 			(effects
@@
 			)
 		)
-		(property "Value" "33k"
+		(property "Value" "24.9k"
 			(at 83.82 27.94 90)
 			(effects
