File: Hardware/g081_audio/g081_audio.kicad_sch (KiCad schematic)
At the start: 29 parts, among them J1 Serial, J2 SWD, U1 12MHz, U11 OLED_I2C, U2 MCP1802x-xx02xOT, U3 STM32G081KB, U4 W25Q32JVSS, U5 PT8211

Commit message: Added schematic and more documentation.
Other:
- note added: "Bridge 3-2 for I2S output."
- note added: "Optional - not needed for MIDIVerb firmware."
Changed lines of the file:
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@@
+		)
+	)
+	(text "Optional - not needed for MIDIVerb firmware."
+		(exclude_from_sim no)
+		(at 331.216 142.748 0)
+		(effects
+			(font
+				(size 1.27 1.27)
+			)
+		)
+	)
+	(text "Bridge 3-2 for I2S output."
+		(exclude_from_sim no)
+		(at 368.808 206.502 0)
+		(effects
+			(font
+				(size 1.27 1.27)
+			)
 		)
 	)

Commit message: Schematic updates - printing prefs, text notes, input gain, BOM.
Other:
- note added: "Bridge 2-3 for I2S output"
- note added: "Optional - not used by MIDIVerb firmware."
- note removed: "Bridge 3-2 for I2S output."
- note removed: "Optional - not needed for MIDIVerb firmware."
Changed lines of the file:
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@@
 		)
 	)
-	(text "Optional - not needed for MIDIVerb firmware."
+	(text "Optional - not used by MIDIVerb firmware."
 		(exclude_from_sim no)
-		(at 331.216 142.748 0)
+		(at 330.2 143.764 0)
 		(effects
 			(font
@@
 		)
 	)
-	(text "Bridge 3-2 for I2S output."
+	(text "Bridge 2-3 for I2S output"
 		(exclude_from_sim no)
-		(at 368.808 206.502 0)
+		(at 389.89 192.278 0)
 		(effects
 			(font
